File: Hardware/PCB/Residential_PCB_Design-SMD/Residential_PCB_Design-SMD.kicad_pcb (KiCad board)
At the start: 2 copper layers, 110 x 60 mm, 44 parts, among them IC1 PCF8523T_1,118, J1 SD_CARD_SOCKET, J2 Screw_Terminal_01x02, J3 Screw_Terminal_01x05, J4 USB_B_Micro, J5 ISP Header, J6 2895, SW1 SW_Push, SW2 SW_Push, SW3 SW_DIP_x02, U1 MCP1703A-3302_SOT23, U2 ATmega328P-AU, U3 FT232RL, Y1 8MHz, Y2 32.768kHz

Commit message: Updating PCB Design
Parts:
- Y1: footprint Crystal:Crystal_SMD_2012-2Pin_2.0x1.2mm_HandSoldering -> Crystal:Crystal_SMD_Abracon_ABM3-2Pin_5.0x3.2mm
- moved C6 3.87 mm to (83.8, 139.1), turned to 270 degrees
- moved Y1 1.85 mm to (86.8, 142.2)
- moved C7 0.82 mm to (83.8, 145.3), turned to 90 degrees
- moved J4 0.09 mm to (52.8, 122.9)
Routing:
- net GND: track 33.7 -> 29.6 mm, vias 4 -> 23
- net Net-(C6-Pad2): track 5.31 -> 7.72 mm
- net Net-(D1-Pad2): track 2.66 -> 4.50 mm
- net Net-(C7-Pad2): track 6.36 -> 7.69 mm
Other:
- board text added: "-+"
- board text added: "PRGRM"
- board text added: "PWR"
- board text added: "RESET"
- board text added: "SENSOR"
- board text added: "SMT Pads: xx Thru Holes: xx Number of unique parts: xx Dimensions: 4.3307 in. by 2.3583 in. OR 109.9998 mm by 59.9008 mm"
- board text added: "USB Power"
- board text added: "WHT BWN GRN GND 3V3"
- board text added: "Wake Up"
