File: Hardware/PCB/Residential_PCB_Design-SMD/Residential_PCB_Design-SMD.sch (KiCad schematic (older format))
At the start: 40 parts, among them IC1 PCF8523T_1,118, J1 SD_CARD_SOCKET, J2 Screw_Terminal_01x02, J3 Screw_Terminal_01x05, J4 USB_B_Micro, J5 ISP Header, J6 2895, SW1 SW_Push, SW2 SW_Push, SW3 SW_DIP_x02, U1 MCP1703A-3302_SOT23, U2 ATmega328P-AU, U3 FT232RL, Y1 8MHz, Y2 32.768kHz

Commit message: Updating PCB Design
Parts:
- Y1: footprint Crystal:Crystal_SMD_2012-2Pin_2.0x1.2mm_HandSoldering -> Crystal:Crystal_SMD_Abracon_ABM3-2Pin_5.0x3.2mm
Changed lines of the file:
@@
 F 0 "Y1" V 5850 3450 50  0000 L CNN
 F 1 "8MHz" V 6050 3350 50  0000 L CNN
-F 2 "Crystal:Crystal_SMD_2012-2Pin_2.0x1.2mm_HandSoldering" H 5900 3400 50  0001 C CNN
+F 2 "Crystal:Crystal_SMD_Abracon_ABM3-2Pin_5.0x3.2mm" H 5900 3400 50  0001 C CNN
 F 3 "~" H 5900 3400 50  0001 C CNN
 	1    5900 3400
